File: hardware/KungFuFlash.kicad_pcb (KiCad board)
At the start: 2 copper layers, 58 x 62 mm, 40 parts, among them J1 USB Power, J2 USB_B_Micro, J4 SWD, Q1 BC817, SW1 Reset, SW2 Menu, SW3 Special, U1 C64-Exp-Port, U2 AMS1117-3.3, U3 STM32F405RGTx, Y1 8MHz

Commit message: PCB rev. 2
Parts:
- moved J2 4.55 mm to (135.6, 86.5)
- moved RN1 3.43 mm to (115.4, 115.8)
- moved RN2 3.43 mm to (125.0, 115.8)
- moved J1 2.42 mm to (122.9, 86.4)
- moved REF** 1.54 mm to (125.4, 110.2)
- moved J4 1.27 mm to (125.4, 94.4)
- moved C10 0.51 mm to (113.1, 109.7)
- moved C12 0.13 mm to (109.5, 112.2)
Routing:
- net GND: track 563.9 -> 751.1 mm, vias 57 -> 66
- net /D7: track 18.7 -> 14.6 mm
- net /D4: track 30.8 -> 26.9 mm
- net /D6: track 20.3 -> 16.3 mm
- net /CD1: track 6.42 -> 10.4 mm
- net /D5: track 29.2 -> 25.6 mm
- net /D3: track 42.5 -> 38.9 mm
- net /CD6: track 6.48 -> 10.0 mm
- net /D0: track 44.6 -> 41.1 mm
- net /CD2: track 6.21 -> 9.64 mm
- net /D1: track 43.5 -> 40.1 mm
- net /CD0: track 8.09 -> 11.3 mm
- net /CD5: track 6.20 -> 9.35 mm
- net /D2: track 42.4 -> 39.3 mm
- net /CD7: track 8.17 -> 11.2 mm
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Other:
- board size 58 x 62 mm -> 60.6 x 62 mm
- board text added: "Rev. 2"
- board text removed: "Rev. 1"
